File: Tubetester03.kicad_pcb (KiCad board)
At the start: 2 copper layers, 24 parts, among them Q1 IRF830, Q2 2N3904

Commit message: Add files via upload
Other:
- net class low current added: clearance 0.2, trace_width 0.5, via_dia 0.6, via_drill 0.4
Changed lines of the file:
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@@
     (thickness 1.6)
     (drawings 2)
-    (tracks 51)
+    (tracks 52)
     (zones 0)
     (modules 24)
@@
     (visible_elements 7FFFFFFF)
     (pcbplotparams
-      (layerselection 0x00030_80000001)
+      (layerselection 0x00000_80000001)
       (usegerberextensions false)
       (excludeedgelayer true)
@@
       (padsonsilk false)
       (subtractmaskfromsilk false)
-      (outputformat 1)
+      (outputformat 5)
       (mirror false)
-      (drillshape 1)
+      (drillshape 0)
       (scaleselection 1)
       (outputdirectory ./))
@@
     (add_net /Vout)
     (add_net GND)
-    (add_net "Net-(C1-Pad1)")
     (add_net "Net-(C5-Pad2)")
     (add_net "Net-(D1-Pad1)")
@@
     (add_net "Net-(R4-Pad1)")
     (add_net "Net-(R5-Pad1)")
+  )
+  (net_class "low current" ""
+    (clearance 0.2)
+    (trace_width 0.5)
+    (via_dia 0.6)
+    (via_drill 0.4)
+    (uvia_dia 0.3)
+    (uvia_drill 0.1)
+    (add_net "Net-(C1-Pad1)")
   )
   (module Capacitors_THT:C_Rect_L16.5mm_W6.0mm_P15.00mm_MKT (layer F.Cu)
@@
     (arrow2b (pts (xy 174.625 67.945) (xy 175.751504 67.358579)))
   )
-  (segment (start 204.47 85.09) (end 204.47 89.535) (width 1) (layer B.Cu) (net 1) (status 400000))
-  (segment (start 204.47 89.535) (end 205.74 90.805) (width 1) (layer B.Cu) (net 1) (status 800000))
-  (segment (start 205.74 90.805) (end 205.74 91.44) (width 1) (layer B.Cu) (net 1) (status C00000))
+  (segment (start 228.6 96.52) (end 218.44 96.52) (width 0.5) (layer B.Cu) (net 1) (status 400000))
+  (segment (start 217.805 97.155) (end 210.82 97.155) (width 0.5) (layer B.Cu) (net 1))
+  (segment (start 218.44 96.52) (end 217.805 97.155) (width 0.5) (layer B.Cu) (net 1))
+  (segment (start 204.47 85.09) (end 204.47 89.535) (width 1) (layer B.Cu) (net 1))
+  (segment (start 204.47 89.535) (end 205.74 90.805) (width 1) (layer B.Cu) (net 1))
+  (segment (start 205.74 90.805) (end 205.74 91.44) (width 1) (layer B.Cu) (net 1))
   (segment (start 200.66 104.14) (end 200.66 101.6) (width 1) (layer B.Cu) (net 1))
   (segment (start 200.66 101.6) (end 207.01 95.25) (width 1) (layer B.Cu) (net 1))
   (segment (start 205.74 91.44) (end 205.74 93.98) (width 1) (layer B.Cu) (net 1))
   (segment (start 205.74 93.98) (end 207.01 95.25) (width 1) (layer B.Cu) (net 1))
-  (segment (start 210.82 97.155) (end 227.965 97.155) (width 1) (layer B.Cu) (net 1))
-  (segment (start 227.965 97.155) (end 228.6 96.52) (width 1) (layer B.Cu) (net 1))
   (segment (start 207.01 95.25) (end 210.82 95.25) (width 1) (layer B.Cu) (net 1))
   (segment (start 210.82 95.25) (end 210.82 97.155) (width 1) (layer B.Cu) (net 1))
   (segment (start 210.82 97.155) (end 210.82 99.06) (width 1) (layer B.Cu) (net 1))
-  (segment (start 195.58 87.63) (end 195.58 86.36) (width 1) (layer B.Cu) (net 2) (status C00000))
-  (segment (start 195.58 86.36) (end 201.93 80.01) (width 1) (layer B.Cu) (net 2) (status C00000))
+  (segment (start 195.58 87.63) (end 195.58 86.36) (width 1) (layer B.Cu) (net 2))
+  (segment (start 195.58 86.36) (end 201.93 80.01) (width 1) (layer B.Cu) (net 2))
   (segment (start 184.15 88.265) (end 180.34 88.265) (width 1) (layer B.Cu) (net 3))
   (segment (start 180.34 88.265) (end 179.07 89.535) (width 1) (layer B.Cu) (net 3))
